File: yts-pcb/yts-pcb.kicad_sch (KiCad schematic)
At the start: 58 parts

Commit message: finish schematics
Connections:
- net col0: now also U?.20 (A3/PF4)
- net col1: now also U?.19 (A2/PF5)
- net col2: now also U?.18 (A1/PF6)
- net col3: now also U?.17 (A0/PF7)
- net col4: now also U?.16 (15/PB1)
- net col5: now also U?.15 (14/PB3)
- net col6: now also U?.14 (16/PB2)
- net row0: now also U?.9 (6/PD7)
- net row1: now also U?.10 (7/PE6)
- net row2: now also U?.11 (8/PB4)
- net row3: now also U?.12 (9/PB5)
- net col7: now reaches U?.13 (10/PB6)
- net GND: now reaches U?.23 (GND)
- net GND: now also U?.3 (GND), U?.4 (GND)
- net BAT: now reaches U?.24 (RAW)
- no-connect marks 1 -> 3

Commit message: finish schematics and footprints
Parts:
- removed D? (x2): DIODE, symbol Simulation_SPICE:DIODE
- removed SW?: MX, symbol Switch:SW_Push
- removed SW?: SW_DPDT_x2, symbol Switch:SW_DPDT_x2
- added D27, D28, D29: DIODE, keebio:Diode-Hybrid-Back, symbol Simulation_SPICE:DIODE
- added J1: B+, Connector_Wire:SolderWirePad_1x01_SMD_1x2mm, symbol Connector:Conn_01x01_Female
- added J2: B-, Connector_Wire:SolderWirePad_1x01_SMD_1x2mm, symbol Connector:Conn_01x01_Female
- added SW1: ON/OFF, Button_Switch_SMD:SW_SPDT_PCM12, symbol Switch:SW_DPDT_x2
- added SW25, SW28: MX, Button_Switch_Keyboard:SW_Cherry_MX_1.00u_PCB, symbol Switch:SW_Push
- D1, D10, D11, D12, D13, D14, D15, D16, D17, D18, D19, D2, D20, D21, D22, D23, D24, D25, D26, D3, D4, D5, D6, D7, D8, D9: renamed from D?; footprint (none) -> keebio:Diode-Hybrid-Back
- SW10, SW11, SW12, SW13, SW14, SW15, SW16, SW17, SW18, SW19, SW2, SW20, SW21, SW22, SW23, SW24, SW26, SW27, SW3, SW4, SW5, SW6, SW7, SW8, SW9: renamed from SW?; footprint (none) -> Button_Switch_Keyboard:SW_Cherry_MX_1.00u_PCB
- SW29, SW30: renamed from SW?; footprint (none) -> keebio:RotaryEncoder_EC11
- U1: renamed from U?; footprint (none) -> keebio:ArduinoProMicro-BackSide
Connections:
- net BAT: now also SW1.1 (A)
- net GND: now also SW29.C, SW30.C, J2.1 (Pin_1)
- net VCC: now also U1.21 (VCC)
- net col6: now also SW25.2; no longer SW29.S2, SW30.S2
- net col7: now also SW29.S2, SW30.S2, SW28.2
- net row0: now also D27.2 (K)
- net row1: now also D28.2 (K)
- net row2: now also D29.2 (K)
- net at SW30.S1: now also D29.1 (A)
- net enc0: now reaches SW29.A
- net enc0: now also U1.5 (2/PD1)
- net enc1: now reaches SW29.B
- net enc1: now also U1.6 (3/PD0)
- net at SW29.S1: now also D27.1 (A); no longer D24.1 (A)
- net enc2: now reaches U1.7 (4/PD4)
- net enc2: now also SW30.A
- net enc3: now reaches U1.8 (5/PC6)
- net enc3: now also SW30.B
- new net: D28.1 (A), SW28.1
- new net: J1.1 (Pin_1), SW1.2 (B)
- new net: D24.1 (A), SW25.1
- no-connect marks 3 -> 4
Other:
- title: (none) -> YTS-Interface 1
- moved on the sheet: SW29, SW30

Commit message: finish pcb layout
Connections:
- net col4: now also SW28.2
- net col7: no longer SW28.2
- net row1: no longer D28.2 (K)
- net row2: now also D28.2 (K)
Changed lines of the file:
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@@
   (junction (at 199.39 38.1) (diameter 0) (color 0 0 0 0)
   )
+  (junction (at 168.91 68.58) (diameter 0) (color 0 0 0 0)
+  )
   (junction (at 153.67 38.1) (diameter 0) (color 0 0 0 0)
   )
@@
   (junction (at 184.15 68.58) (diameter 0) (color 0 0 0 0)
   )
+  (junction (at 158.75 76.2) (diameter 0) (color 0 0 0 0)
+  )
   (junction (at 99.06 91.44) (diameter 0) (color 0 0 0 0)
   )
@@
   (junction (at 173.99 45.72) (diameter 0) (color 0 0 0 0)
   )
-  (junction (at 189.23 60.96) (diameter 0) (color 0 0 0 0)
-  )
   (junction (at 124.46 68.58) (diameter 0) (color 0 0 0 0)
   )
@@
   )
   (junction (at 214.63 33.02) (diameter 0) (color 0 0 0 0)
-  )
-  (junction (at 214.63 53.34) (diameter 0) (color 0 0 0 0)
   )
   (junction (at 129.54 91.44) (diameter 0) (color 0 0 0 0)
@@
     (stroke (width 0) (type default) (color 0 0 0 0))
   )
-  (wire (pts (xy 214.63 33.02) (xy 214.63 53.34))
+  (wire (pts (xy 158.75 76.2) (xy 173.99 76.2))
     (stroke (width 0) (type default) (color 0 0 0 0))
   )
@@
     (stroke (width 0) (type default) (color 0 0 0 0))
   )
-  (wire (pts (xy 189.23 60.96) (xy 204.47 60.96))
-    (stroke (width 0) (type default) (color 0 0 0 0))
-  )
   (wire (pts (xy 214.63 33.02) (xy 219.71 33.02))
     (stroke (width 0) (type default) (color 0 0 0 0))
@@
     (stroke (width 0) (type default) (color 0 0 0 0))
   )
-  (wire (pts (xy 168.91 53.34) (xy 168.91 83.82))
+  (wire (pts (xy 168.91 53.34) (xy 168.91 68.58))
     (stroke (width 0) (type default) (color 0 0 0 0))
   )
@@
     (stroke (width 0) (type default) (color 0 0 0 0))
   )
-  (wire (pts (xy 214.63 63.5) (xy 214.63 53.34))
+  (wire (pts (xy 214.63 33.02) (xy 214.63 63.5))
     (stroke (width 0) (type default) (color 0 0 0 0))
   )
@@
     (stroke (width 0) (type default) (color 0 0 0 0))
   )
+  (wire (pts (xy 168.91 68.58) (xy 168.91 83.82))
+    (stroke (width 0) (type default) (color 0 0 0 0))
+  )
   (wire (pts (xy 219.71 63.5) (xy 214.63 63.5))
     (stroke (width 0) (type default) (color 0 0 0 0))
@@
     (stroke (width 0) (type default) (color 0 0 0 0))
   )
-  (wire (pts (xy 143.51 76.2) (xy 173.99 76.2))
+  (wire (pts (xy 143.51 76.2) (xy 158.75 76.2))
     (stroke (width 0) (type default) (color 0 0 0 0))
   )
@@
     (property "Datasheet" "~" (id 3) (at 104.14 33.02 0)
       (effects (font (size 1.27 1.27)) hide)
-    )
-    (pin "1")
-    (pin "2")
-  )
-  (symbol (lib_id "Simulation_SPICE:DIODE") (at 204.47 57.15 270) (unit 1)
-    (in_bom yes) (on_board yes) (fields_autoplaced)
-    (property "Reference" "D28" (id 0) (at 210.82 57.15 0)
-      (effects (font (size 1.27 1.27)) hide)
-    )
-    (property "Value" "DIODE" (id 1) (at 207.01 57.785 90)
-      (effects (font (size 1 1)) (justify left))
-    )
-    (property "Footprint" "keebio:Diode-Hybrid-Back" (id 2) (at 204.47 57.15 0)
-      (effects (font (size 1.27 1.27)) hide)
-    )
-    (property "Datasheet" "~" (id 3) (at 204.47 57.15 0)
-      (effects (font (size 1.27 1.27)) hide)
-    )
-    (property "Spice_Netlist_Enabled" "Y" (id 4) (at 204.47 57.15 0)
-      (effects (font (size 1.27 1.27)) (justify left) hide)
-    )
-    (property "Spice_Primitive" "D" (id 5) (at 204.47 57.15 0)
-      (effects (font (size 1.27 1.27)) (justify left) hide)
     )
     (pin "1")
@@
     (pin "2")
   )
+  (symbol (lib_id "Simulation_SPICE:DIODE") (at 158.75 72.39 270) (unit 1)
+    (in_bom yes) (on_board yes) (fields_autoplaced)
+    (property "Reference" "D28" (id 0) (at 165.1 72.39 0)
+      (effects (font (size 1.27 1.27)) hide)
+    )
+    (property "Value" "DIODE" (id 1) (at 161.29 73.025 90)
+      (effects (font (size 1 1)) (justify left))
+    )
+    (property "Footprint" "keebio:Diode-Hybrid-Back" (id 2) (at 158.75 72.39 0)
+      (effects (font (size 1.27 1.27)) hide)
+    )
+    (property "Datasheet" "~" (id 3) (at 158.75 72.39 0)
+      (effects (font (size 1.27 1.27)) hide)
+    )
+    (property "Spice_Netlist_Enabled" "Y" (id 4) (at 158.75 72.39 0)
+      (effects (font (size 1.27 1.27)) (justify left) hide)
+    )
+    (property "Spice_Primitive" "D" (id 5) (at 158.75 72.39 0)
+      (effects (font (size 1.27 1.27)) (justify left) hide)
+    )
+    (pin "1")
+    (pin "2")
+  )
   (symbol (lib_id "Device:RotaryEncoder_Switch") (at 227.33 66.04 180) (unit 1)
     (in_bom yes) (on_board yes)
@@
     (pin "6")
   )
+  (symbol (lib_id "Switch:SW_Push") (at 163.83 68.58 0) (unit 1)
+    (in_bom yes) (on_board yes) (fields_autoplaced)
+    (property "Reference" "SW28" (id 0) (at 163.83 63.5 0)
+      (effects (font (size 1 1)) (justify top))
+    )
+    (property "Value" "MX" (id 1) (at 163.83 63.5 0)
+      (effects (font (size 1 1)) (justify bottom))
+    )
+    (property "Footprint" "Button_Switch_Keyboard:SW_Cherry_MX_1.00u_PCB" (id 2) (at 163.83 63.5 0)
+      (effects (font (size 1.27 1.27)) hide)
+    )
+    (property "Datasheet" "~" (id 3) (at 163.83 63.5 0)
+      (effects (font (size 1.27 1.27)) hide)
+    )
+    (pin "1")
+    (pin "2")
+  )
   (symbol (lib_id "Simulation_SPICE:DIODE") (at 189.23 41.91 270) (unit 1)
     (in_bom yes) (on_board yes) (fields_autoplaced)
@@
     )
     (property "Datasheet" "~" (id 3) (at 179.07 78.74 0)
-      (effects (font (size 1.27 1.27)) hide)
-    )
-    (pin "1")
-    (pin "2")
-  )
-  (symbol (lib_id "Switch:SW_Push") (at 209.55 53.34 0) (unit 1)
-    (in_bom yes) (on_board yes) (fields_autoplaced)
-    (property "Reference" "SW28" (id 0) (at 209.55 48.26 0)
-      (effects (font (size 1 1)) (justify top))
-    )
-    (property "Value" "MX" (id 1) (at 209.55 48.26 0)
-      (effects (font (size 1 1)) (justify bottom))
-    )
-    (property "Footprint" "Button_Switch_Keyboard:SW_Cherry_MX_1.00u_PCB" (id 2) (at 209.55 48.26 0)
-      (effects (font (size 1.27 1.27)) hide)
-    )
-    (property "Datasheet" "~" (id 3) (at 209.55 48.26 0)
       (effects (font (size 1.27 1.27)) hide)
     )
@@
       (reference "D27") (unit 1) (value "DIODE") (footprint "keebio:Diode-Hybrid-Back")
     )
-    (path "/0af7a86a-155f-4cb8-97a3-8ed2b2c722e4"
+    (path "/c035d932-fda2-4019-8089-96b1e49d1b88"
       (reference "D28") (unit 1) (value "DIODE") (footprint "keebio:Diode-Hybrid-Back")
     )
@@
       (reference "SW27") (unit 1) (value "MX") (footprint "Button_Switch_Keyboard:SW_Cherry_MX_1.00u_PCB")
     )
-    (path "/fa5ff19d-6a75-41d0-ac94-98bd5a3f0db0"
+    (path "/ca1cb953-4fc1-4d33-8320-283bf74a730a"
       (reference "SW28") (unit 1) (value "MX") (footprint "Button_Switch_Keyboard:SW_Cherry_MX_1.00u_PCB")
     )

Commit message: update mx switches footprints to plate mount
Parts:
- SW10, SW11, SW12, SW13, SW14, SW15, SW16, SW17, SW18, SW19, SW2, SW20, SW21, SW22, SW23, SW24, SW25, SW26, SW27, SW28, SW3, SW4, SW5, SW6, SW7, SW8, SW9: footprint Button_Switch_Keyboard:SW_Cherry_MX_1.00u_PCB -> Button_Switch_Keyboard:SW_Cherry_MX_1.00u_Plate

Commit message: update footprints
Parts:
- SW10, SW11, SW12, SW13, SW14, SW15, SW16, SW17, SW18, SW19, SW2, SW20, SW21, SW22, SW23, SW24, SW25, SW26, SW27, SW28, SW3, SW4, SW5, SW6, SW7, SW8, SW9: footprint Button_Switch_Keyboard:SW_Cherry_MX_1.00u_Plate -> Button_Switch_Keyboard:SW_Cherry_MX_1.00u_PCB
