File: yts-pcb/yts-pcb.kicad_pcb (KiCad board)
At the start: 2 copper layers, 210 x 78 mm, 62 parts, among them J1 B+, J2 B-, SW1 ON/OFF, SW10 MX, SW11 MX, SW12 MX, SW13 MX, SW14 MX, SW15 MX, SW16 MX, SW17 MX, SW18 MX, SW19 MX, SW2 MX, SW20 MX, SW21 MX, SW22 MX, SW23 MX, SW24 MX, SW25 MX, SW26 MX, SW27 MX, SW28 MX, SW29 RotaryEncoder_Switch, SW3 MX, SW30 RotaryEncoder_Switch, SW4 MX, SW5 MX, SW6 MX, SW7 MX, SW8 MX, SW9 MX, U1 Nice!Nano

Commit message: update footprints
Parts:
- SW10, SW11, SW12, SW13, SW14, SW15, SW16, SW17, SW18, SW19, SW2, SW20, SW21, SW22, SW23, SW24, SW25, SW26, SW27, SW28, SW3, SW4, SW5, SW6, SW7, SW8, SW9: footprint Button_Switch_Keyboard:SW_Cherry_MX_1.00u_Plate -> Button_Switch_Keyboard:SW_Cherry_MX_1.00u_PCB
Routing:
- added copper zone on B.Cu, net GND
- added copper zone on F.Cu, net GND

Commit message: make gerbers rev0
Other:
- board text added: "yts-1 rev0"
Changed lines of the file:
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@@
   (gr_rect (start 82 83) (end 95 96) (layer "User.1") (width 0.15) (fill none))
   (gr_rect (start 82 64) (end 95 77) (layer "User.1") (width 0.15) (fill none))
+  (gr_text "yts-1 rev0" (at 225 45) (layer "B.SilkS")
+    (effects (font (size 1.5 1.5) (thickness 0.3)) (justify mirror))
+  )
+  (gr_text "yts-1 rev0" (at 223 45) (layer "F.SilkS")
+    (effects (font (size 1.5 1.5) (thickness 0.3)))
+  )
   (segment (start 128.5 49) (end 123.4713 54.0287) (width 0.25) (layer "F.Cu") (net 1))
   (segment (start 123.4713 54.0287) (end 117.8713 54.0287) (width 0.25) (layer "F.Cu") (net 1))
