File: yts-pcb/yts-pcb.kicad_pcb (KiCad board)
At the start: 2 copper layers, 285 x 94 mm, 67 parts, among them J1 B+, J2 B-, SW1 ON/OFF, SW10 MX, SW11 MX, SW12 MX, SW13 MX, SW14 MX, SW15 MX, SW16 MX, SW17 MX, SW18 MX, SW19 MX, SW2 MX, SW20 MX, SW21 MX, SW22 MX, SW23 MX, SW24 MX, SW25 MX, SW26 MX, SW27 MX, SW28 MX, SW29 RotaryEncoder_Switch, SW3 MX, SW30 RotaryEncoder_Switch, SW4 MX, SW5 MX, SW6 MX, SW7 MX, SW8 MX, SW9 MX, U1 Nice!Nano

Commit message: finish rev1
Parts:
- removed the REF** at (212.5, 108.5)
- moved REF** 76.3 mm to (66.0, 144.8)
- moved REF** 76.3 mm to (87.2, 116.2)
- moved REF** 76.3 mm to (322.0, 116.2)
- moved REF** 76.3 mm to (343.0, 144.8)
- moved D27 75.2 mm to (302.1, 115.2)
- moved D13 75.2 mm to (179.0, 106.2)
- moved D14 75.2 mm to (179.0, 125.7)
- moved D17 75.2 mm to (236.0, 106.2)
- moved D18 75.2 mm to (236.0, 125.7)
- moved D20 75.2 mm to (255.0, 106.2)
- moved D21 75.2 mm to (255.0, 125.7)
- moved D23 75.2 mm to (255.0, 163.8)
- moved D24 75.2 mm to (274.0, 106.2)
- moved D25 75.2 mm to (274.0, 125.7)
- moved J1 75.2 mm to (210.0, 106.2)
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Other:
- outline, holes or cut-outs redrawn
- board text added: "yts-1 rev1"
- board text removed: "yts-1 rev0"

Commit message: add 3d models for presentation
Parts:
- added REF**: KBDFans Tofu60, MountingEquipment:KBDFans Tofu60, F.Cu at (206.0, 234.0)
Other:
- board size 285 x 94 mm -> 287 x 96.6 mm
