File: yts-switchblade/yts-switchblade.kicad_pcb (KiCad board)
At the start: 2 copper layers, 248 x 116 mm, 4 parts

Commit message: make gerbers rev0
Parts:
- removed the REF** at (26.5, 144.0)
- removed the REF** at (26.5, 34.0)
- removed the REF** at (268.5, 34.0)
- removed the REF** at (268.5, 144.0)
- added REF**: MountingHole_2.2mm_M2, MountingHole:MountingHole_2.2mm_M2, F.Cu at (268.5, 144.0)
- added REF**: MountingHole_2.2mm_M2, MountingHole:MountingHole_2.2mm_M2, F.Cu at (268.5, 34.0)
- added REF**: MountingHole_2.2mm_M2, MountingHole:MountingHole_2.2mm_M2, F.Cu at (26.5, 34.0)
- added REF**: MountingHole_2.2mm_M2, MountingHole:MountingHole_2.2mm_M2, F.Cu at (26.5, 144.0)
Routing:
- added copper zone on B.Cu, net (none)
- added copper zone on F.Cu, net (none)
Other:
- board text added: "PROTOTYPE – FOR TESTING PURPOSES ONLY"
- board text added: "yts-1"
Changed lines of the file:
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@@
       (layerselection 0x00010fc_ffffffff)
       (disableapertmacros false)
-      (usegerberextensions false)
+      (usegerberextensions true)
       (usegerberattributes true)
       (usegerberadvancedattributes true)
@@
       (plotinvisibletext false)
       (sketchpadsonfab false)
-      (subtractmaskfromsilk false)
+      (subtractmaskfromsilk true)
       (outputformat 1)
       (mirror false)
-      (drillshape 1)
+      (drillshape 0)
       (scaleselection 1)
-      (outputdirectory "")
+      (outputdirectory "yts-switchblade-gerbers-rev0/")
     )
   )
   (net 0 "")
-  (footprint "MountingHole:MountingHole_2.5mm" (layer "F.Cu")
-    (at 26.5 144)
-    (descr "Mounting Hole 2.5mm, no annular")
-    (tags "mounting hole 2.5mm no annular")
+  (footprint "MountingHole:MountingHole_2.2mm_M2" (layer "F.Cu")
+    (at 268.5 144)
+    (descr "Mounting Hole 2.2mm, no annular, M2")
+    (tags "mounting hole 2.2mm no annular m2")
     (attr exclude_from_pos_files exclude_from_bom)
-    (fp_text reference "REF**" (at 0 -3.5) (layer "F.SilkS") hide
+    (fp_text reference "REF**" (at 0 -3.2) (layer "F.SilkS") hide
       (effects (font (size 1 1) (thickness 0.15)))
     )
-    (fp_text value "MountingHole_2.5mm" (at 0 3.5) (layer "F.Fab")
+    (fp_text value "MountingHole_2.2mm_M2" (at 0 3.2) (layer "F.Fab")
       (effects (font (size 1 1) (thickness 0.15)))
     )
@@
       (effects (font (size 1 1) (thickness 0.15)))
     )
-    (fp_circle (center 0 0) (end 2.5 0) (layer "Cmts.User") (width 0.15) (fill none))
-    (fp_circle (center 0 0) (end 2.75 0) (layer "F.CrtYd") (width 0.05) (fill none))
-    (pad "" np_thru_hole circle (at 0 0) (size 2.5 2.5) (drill 2.5) (layers *.Cu *.Mask))
+    (fp_circle (center 0 0) (end 2.2 0) (layer "Cmts.User") (width 0.15) (fill none))
+    (fp_circle (center 0 0) (end 2.45 0) (layer "F.CrtYd") (width 0.05) (fill none))
+    (pad "" np_thru_hole circle (at 0 0) (size 2.2 2.2) (drill 2.2) (layers *.Cu *.Mask))
   )
-  (footprint "MountingHole:MountingHole_2.5mm" (layer "F.Cu")
-    (at 26.5 34)
-    (descr "Mounting Hole 2.5mm, no annular")
-    (tags "mounting hole 2.5mm no annular")
+  (footprint "MountingHole:MountingHole_2.2mm_M2" (layer "F.Cu")
+    (at 268.5 34)
+    (descr "Mounting Hole 2.2mm, no annular, M2")
+    (tags "mounting hole 2.2mm no annular m2")
     (attr exclude_from_pos_files exclude_from_bom)
-    (fp_text reference "REF**" (at 0 -3.5) (layer "F.SilkS") hide
+    (fp_text reference "REF**" (at 0 -3.2) (layer "F.SilkS") hide
       (effects (font (size 1 1) (thickness 0.15)))
     )
-    (fp_text value "MountingHole_2.5mm" (at 0 3.5) (layer "F.Fab")
+    (fp_text value "MountingHole_2.2mm_M2" (at 0 3.2) (layer "F.Fab")
       (effects (font (size 1 1) (thickness 0.15)))
     )
@@
       (effects (font (size 1 1) (thickness 0.15)))
     )
-    (fp_circle (center 0 0) (end 2.5 0) (layer "Cmts.User") (width 0.15) (fill none))
-    (fp_circle (center 0 0) (end 2.75 0) (layer "F.CrtYd") (width 0.05) (fill none))
-    (pad "" np_thru_hole circle (at 0 0) (size 2.5 2.5) (drill 2.5) (layers *.Cu *.Mask))
+    (fp_circle (center 0 0) (end 2.2 0) (layer "Cmts.User") (width 0.15) (fill none))
+    (fp_circle (center 0 0) (end 2.45 0) (layer "F.CrtYd") (width 0.05) (fill none))
+    (pad "" np_thru_hole circle (at 0 0) (size 2.2 2.2) (drill 2.2) (layers *.Cu *.Mask))
   )
-  (footprint "MountingHole:MountingHole_2.5mm" (layer "F.Cu")
-    (at 268.5 34)
-    (descr "Mounting Hole 2.5mm, no annular")
-    (tags "mounting hole 2.5mm no annular")
+  (footprint "MountingHole:MountingHole_2.2mm_M2" (layer "F.Cu")
+    (at 26.5 34)
+    (descr "Mounting Hole 2.2mm, no annular, M2")
+    (tags "mounting hole 2.2mm no annular m2")
     (attr exclude_from_pos_files exclude_from_bom)
-    (fp_text reference "REF**" (at 0 -3.5) (layer "F.SilkS") hide
+    (fp_text reference "REF**" (at 0 -3.2) (layer "F.SilkS") hide
       (effects (font (size 1 1) (thickness 0.15)))
     )
-    (fp_text value "MountingHole_2.5mm" (at 0 3.5) (layer "F.Fab")
+    (fp_text value "MountingHole_2.2mm_M2" (at 0 3.2) (layer "F.Fab")
       (effects (font (size 1 1) (thickness 0.15)))
     )
@@
       (effects (font (size 1 1) (thickness 0.15)))
     )
-    (fp_circle (center 0 0) (end 2.5 0) (layer "Cmts.User") (width 0.15) (fill none))
-    (fp_circle (center 0 0) (end 2.75 0) (layer "F.CrtYd") (width 0.05) (fill none))
-    (pad "" np_thru_hole circle (at 0 0) (size 2.5 2.5) (drill 2.5) (layers *.Cu *.Mask))
+    (fp_circle (center 0 0) (end 2.2 0) (layer "Cmts.User") (width 0.15) (fill none))
+    (fp_circle (center 0 0) (end 2.45 0) (layer "F.CrtYd") (width 0.05) (fill none))
+    (pad "" np_thru_hole circle (at 0 0) (size 2.2 2.2) (drill 2.2) (layers *.Cu *.Mask))
   )
-  (footprint "MountingHole:MountingHole_2.5mm" (layer "F.Cu")
-    (at 268.5 144)
-    (descr "Mounting Hole 2.5mm, no annular")
-    (tags "mounting hole 2.5mm no annular")
+  (footprint "MountingHole:MountingHole_2.2mm_M2" (layer "F.Cu")
+    (at 26.5 144)
+    (descr "Mounting Hole 2.2mm, no annular, M2")
+    (tags "mounting hole 2.2mm no annular m2")
     (attr exclude_from_pos_files exclude_from_bom)
-    (fp_text reference "REF**" (at 0 -3.5) (layer "F.SilkS") hide
+    (fp_text reference "REF**" (at 0 -3.2) (layer "F.SilkS") hide
       (effects (font (size 1 1) (thickness 0.15)))
     )
-    (fp_text value "MountingHole_2.5mm" (at 0 3.5) (layer "F.Fab")
+    (fp_text value "MountingHole_2.2mm_M2" (at 0 3.2) (layer "F.Fab")
       (effects (font (size 1 1) (thickness 0.15)))
     )
@@
       (effects (font (size 1 1) (thickness 0.15)))
     )
-    (fp_circle (center 0 0) (end 2.5 0) (layer "Cmts.User") (width 0.15) (fill none))
-    (fp_circle (center 0 0) (end 2.75 0) (layer "F.CrtYd") (width 0.05) (fill none))
-    (pad "" np_thru_hole circle (at 0 0) (size 2.5 2.5) (drill 2.5) (layers *.Cu *.Mask))
+    (fp_circle (center 0 0) (end 2.2 0) (layer "Cmts.User") (width 0.15) (fill none))
+    (fp_circle (center 0 0) (end 2.45 0) (layer "F.CrtYd") (width 0.05) (fill none))
+    (pad "" np_thru_hole circle (at 0 0) (size 2.2 2.2) (drill 2.2) (layers *.Cu *.Mask))
   )
   (gr_rect (start 179.5 73) (end 192.5 86) (layer "Edge.Cuts") (width 0.15) (fill none))
@@
   (gr_rect (start 84.5 73) (end 97.5 86) (layer "Edge.Cuts") (width 0.15) (fill none))
   (gr_rect (start 65.5 92) (end 78.5 105) (layer "Edge.Cuts") (width 0.15) (fill none))
+  (gr_text "PROTOTYPE – FOR TESTING PURPOSES ONLY" (at 32 60 90) (layer "F.SilkS")
+    (effects (font (size 1 1) (thickness 0.15)))
+  )
+  (gr_text "PROTOTYPE – FOR TESTING PURPOSES ONLY" (at 241 136) (layer "F.SilkS")
+    (effects (font (size 1 1) (thickness 0.15)))
+  )
+  (gr_text "PROTOTYPE – FOR TESTING PURPOSES ONLY" (at 241 41) (layer "F.SilkS")
+    (effects (font (size 1 1) (thickness 0.15)))
+  )
+  (gr_text "PROTOTYPE – FOR TESTING PURPOSES ONLY" (at 51 41) (layer "F.SilkS")
+    (effects (font (size 1 1) (thickness 0.15)))
+  )
+  (gr_text "PROTOTYPE – FOR TESTING PURPOSES ONLY" (at 260 60 270) (layer "F.SilkS")
+    (effects (font (size 1 1) (thickness 0.15)))
+  )
+  (gr_text "PROTOTYPE – FOR TESTING PURPOSES ONLY" (at 32 117 90) (layer "F.SilkS")
+    (effects (font (size 1 1) (thickness 0.15)))
+  )
+  (gr_text "yts-1" (at 147.5 42) (layer "F.SilkS")
+    (effects (font (size 1 1) (thickness 0.15)))
+  )
+  (gr_text "PROTOTYPE – FOR TESTING PURPOSES ONLY" (at 260 117 270) (layer "F.SilkS")
+    (effects (font (size 1 1) (thickness 0.15)))
+  )
+  (gr_text "PROTOTYPE – FOR TESTING PURPOSES ONLY" (at 51 136) (layer "F.SilkS")
+    (effects (font (size 1 1) (thickness 0.15)))
+  )
   (via (at 211.9 124.4) (size 0.8) (drill 0.4) (layers "F.Cu" "B.Cu") (free) (net 0))
   (via (at 46.1 124.4) (size 0.8) (drill 0.4) (layers "F.Cu" "B.Cu") (free) (net 0))
@@
   (via (at 211.9 53.6) (size 0.8) (drill 0.4) (layers "F.Cu" "B.Cu") (free) (net 0))
   (via (at 211.9 124.4) (size 0.8) (drill 0.4) (layers "F.Cu" "B.Cu") (free) (net 0))
+  (zone (net 0) (net_name "") (layers F&B.Cu) (hatch edge 0.508)
+    (connect_pads yes (clearance 0.508))
+    (min_thickness 0.254) (filled_areas_thickness no)
+    (fill yes (thermal_gap 0.508) (thermal_bridge_width 0.508) (island_removal_mode 1) (island_area_min 0))
+    (polygon
+      (pts
+        (xy 272.5 30)
+        (xy 272.5 148)
+        (xy 20.5 148)
+        (xy 21.5 29)
+      )
+    )
+  )
 )

Commit message: fix dimensions
Parts:
- removed REF** (x4): MountingHole_2.2mm_M2, MountingHole:MountingHole_2.2mm_M2
Other:
- board size 248 x 116 mm -> 287 x 96.6 mm
- board text removed: "PROTOTYPE – FOR TESTING PURPOSES ONLY"

Commit message: finish rev1
Routing:
- net (no net): vias 6 -> 0
Other:
- outline, holes or cut-outs redrawn

Commit message: fix switchplate rev1 dimensions
Other:
- board size 287 x 96.6 mm -> 286 x 96 mm
