File: yts-switchblade/yts-switchblade.kicad_pcb (KiCad board)
At the start: 2 copper layers, 286 x 96 mm, 0 parts

Commit message: update dimensions
Other:
- outline, holes or cut-outs redrawn
- board text removed: "yts-1"

Commit message: fix height
Other:
- board size 286 x 96 mm -> 286 x 95.6 mm
Changed lines of the file:
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@@
   (net 0 "")
   (gr_rect (start 221.6 66.5) (end 235.6 80.5) (layer "Edge.Cuts") (width 0.15) (fill none))
-  (gr_line (start 330.1 128.9) (end 330.1 36.7) (layer "Edge.Cuts") (width 0.1))
+  (gr_line (start 330.1 128.5) (end 330.1 36.9) (layer "Edge.Cuts") (width 0.1))
   (gr_rect (start 288.5 48) (end 301.5 61) (layer "Edge.Cuts") (width 0.15) (fill none))
-  (gr_line (start 44.1 36.7) (end 44.1 128.7) (layer "Edge.Cuts") (width 0.1))
-  (gr_line (start 328.1 34.7) (end 46.1 34.7) (layer "Edge.Cuts") (width 0.1))
+  (gr_line (start 44.1 36.9) (end 44.1 128.5) (layer "Edge.Cuts") (width 0.1))
+  (gr_line (start 328.1 34.9) (end 46.1 34.9) (layer "Edge.Cuts") (width 0.1))
   (gr_rect (start 221.6 47.5) (end 235.6 61.5) (layer "Edge.Cuts") (width 0.15) (fill none))
   (gr_rect (start 202.6 66.5) (end 216.6 80.5) (layer "Edge.Cuts") (width 0.15) (fill none))
@@
   (gr_rect (start 88.6 104.5) (end 102.6 118.5) (layer "Edge.Cuts") (width 0.15) (fill none))
   (gr_rect (start 107.6 66.5) (end 121.6 80.5) (layer "Edge.Cuts") (width 0.15) (fill none))
-  (gr_line (start 46.1 130.7) (end 328.1 130.7) (layer "Edge.Cuts") (width 0.1))
+  (gr_line (start 46.1 130.5) (end 328.1 130.5) (layer "Edge.Cuts") (width 0.1))
   (gr_rect (start 88.6 66.5) (end 102.6 80.5) (layer "Edge.Cuts") (width 0.15) (fill none))
   (gr_rect (start 240.6 104.5) (end 254.6 118.5) (layer "Edge.Cuts") (width 0.15) (fill none))
   (gr_rect (start 145.6 85.5) (end 159.6 99.5) (layer "Edge.Cuts") (width 0.15) (fill none))
-  (gr_arc (start 44.1 36.7) (mid 44.685786 35.285786) (end 46.1 34.7) (layer "Edge.Cuts") (width 0.1))
-  (gr_arc (start 328.1 34.7) (mid 329.514214 35.285786) (end 330.1 36.7) (layer "Edge.Cuts") (width 0.1))
+  (gr_arc (start 44.1 36.9) (mid 44.685786 35.485786) (end 46.1 34.9) (layer "Edge.Cuts") (width 0.1))
+  (gr_arc (start 328.1 34.9) (mid 329.514214 35.485786) (end 330.1 36.9) (layer "Edge.Cuts") (width 0.1))
   (gr_rect (start 145.6 104.5) (end 159.6 118.5) (layer "Edge.Cuts") (width 0.15) (fill none))
   (gr_rect (start 126.6 47.5) (end 140.6 61.5) (layer "Edge.Cuts") (width 0.15) (fill none))
@@
   (gr_rect (start 174.1 104.5) (end 188.1 118.5) (layer "Edge.Cuts") (width 0.15) (fill none))
   (gr_rect (start 145.6 47.5) (end 159.6 61.5) (layer "Edge.Cuts") (width 0.15) (fill none))
-  (gr_arc (start 46.1 130.7) (mid 44.685786 130.114214) (end 44.1 128.7) (layer "Edge.Cuts") (width 0.1))
+  (gr_arc (start 46.1 130.5) (mid 44.685786 129.914214) (end 44.1 128.5) (layer "Edge.Cuts") (width 0.1))
   (gr_rect (start 107.6 104.5) (end 121.6 118.5) (layer "Edge.Cuts") (width 0.15) (fill none))
   (gr_rect (start 107.6 47.5) (end 121.6 61.5) (layer "Edge.Cuts") (width 0.15) (fill none))
@@
   (gr_rect (start 240.6 47.5) (end 254.6 61.5) (layer "Edge.Cuts") (width 0.15) (fill none))
   (gr_rect (start 88.6 47.5) (end 102.6 61.5) (layer "Edge.Cuts") (width 0.15) (fill none))
-  (gr_arc (start 330.1 128.7) (mid 329.514214 130.114214) (end 328.1 130.7) (layer "Edge.Cuts") (width 0.1))
+  (gr_arc (start 330.1 128.5) (mid 329.514214 129.914214) (end 328.1 130.5) (layer "Edge.Cuts") (width 0.1))
   (gr_rect (start 221.6 85.5) (end 235.6 99.5) (layer "Edge.Cuts") (width 0.15) (fill none))
   (gr_rect (start 202.6 47.5) (end 216.6 61.5) (layer "Edge.Cuts") (width 0.15) (fill none))
@@
   )
   (dimension (type aligned) (layer "User.4")
-    (pts (xy 328.1 130.7) (xy 328.1 34.7))
+    (pts (xy 328.1 130.5) (xy 328.1 34.9))
     (height 10.5)
-    (gr_text "96.0000 mm" (at 337.45 82.7 90) (layer "User.4")
+    (gr_text "95.6000 mm" (at 337.45 82.7 90) (layer "User.4")
       (effects (font (size 1 1) (thickness 0.15)))
     )
@@
   )
   (dimension (type aligned) (layer "User.4")
-    (pts (xy 44.1 36.7) (xy 330.1 36.7))
+    (pts (xy 44.1 36.9) (xy 330.1 36.9))
     (height -14.7)
-    (gr_text "286.0000 mm" (at 187.1 20.85) (layer "User.4")
+    (gr_text "286.0000 mm" (at 187.1 21.05) (layer "User.4")
       (effects (font (size 1 1) (thickness 0.15)))
     )
