File: yts-switchblade/yts-switchblade.kicad_pcb (KiCad board)
At the start: 2 copper layers, 286 x 95.6 mm, 0 parts

Commit message: add gerbers rev2
Parts:
- added G***: LOGO, LOGO, F.Cu at (66.6, 50.7)
- added G***: LOGO, LOGO, B.Cu at (316.7, 122.3)
